File: PCB/main/chu_main.kicad_pcb (KiCad board)
At the start: 2 copper layers, 294 x 100 mm, 112 parts, among them J1 Conn_01x04, K1 Conn_01x01_Female, K10 Conn_01x01_Female, K11 Conn_01x01_Female, K12 Conn_01x01_Female, K13 Conn_01x01_Female, K14 Conn_01x01_Female, K15 Conn_01x01_Female, K16 Conn_01x01_Female, K17 Conn_01x01_Female, K18 Conn_01x01_Female, K19 Conn_01x01_Female, K2 Conn_01x01_Female, K20 Conn_01x01_Female, K21 Conn_01x01_Female, K22 Conn_01x01_Female, K23 Conn_01x01_Female, K24 Conn_01x01_Female, K25 Conn_01x01_Female, K26 Conn_01x01_Female, K27 Conn_01x01_Female, K28 Conn_01x01_Female, K29 Conn_01x01_Female, K3 Conn_01x01_Female, K30 Conn_01x01_Female, K31 Conn_01x01_Female, K32 Conn_01x01_Female, K4 Conn_01x01_Female, K5 Conn_01x01_Female, K6 Conn_01x01_Female, K7 Conn_01x01_Female, K8 Conn_01x01_Female, K9 Conn_01x01_Female, U0 ChuAcrylic, U1 Pico, U2 PCA9548APW, U3 MPR121QR2_BOARD, U4 MPR121QR2_BOARD, U5 MPR121QR2_BOARD, U8 SN74LV1T34DBV, X1 GP2Y0E03_REAL, X2 GP2Y0E03_REAL, X3 GP2Y0E03_REAL, X4 GP2Y0E03_REAL, X5 GP2Y0E03_REAL

Commit message: wip full size pcb with hc-sr04 ultrasonic sensors
Parts:
- removed IR1, IR2, IR3, IR4, IR5: Conn_01x06, chu_main:GP2Y0E03
- removed J1: Conn_01x04, chu_main:PN532
- removed R10, R11, R12, R13, R4, R5, R6, R7, R8, R9: 4.7K, Resistor_SMD:R_0603_1608Metric
- removed R3: 10, Resistor_SMD:R_0603_1608Metric
- removed U0: ChuAcrylic, chu_main:ChuAcrylic
- removed X1, X2, X3, X4, X5: GP2Y0E03_REAL, chu_main:GP2Y0E03_REAL
- added C10: 0.1uF, Capacitor_SMD:C_0603_1608Metric_Pad1.08x0.95mm_HandSolder, B.Cu at (442.3, 95.8)
- added C11: 0.1uF, Capacitor_SMD:C_0603_1608Metric_Pad1.08x0.95mm_HandSolder, B.Cu at (485.6, 95.8)
- added C9: 0.1uF, Capacitor_SMD:C_0603_1608Metric_Pad1.08x0.95mm_HandSolder, B.Cu at (399.0, 95.8)
- added D37: 1N4148, Diode_THT:D_DO-35_SOD27_P7.62mm_Horizontal, F.Cu at (101.2, 87.4)
- added D38: 1N4148, Diode_THT:D_DO-35_SOD27_P7.62mm_Horizontal, F.Cu at (158.7, 87.4)
- added D39: 1N4148, Diode_THT:D_DO-35_SOD27_P7.62mm_Horizontal, F.Cu at (216.2, 87.4)
- added D40: 1N4148, Diode_THT:D_DO-35_SOD27_P7.62mm_Horizontal, F.Cu at (273.7, 87.4)
- added D41: 1N4148, Diode_THT:D_DO-35_SOD27_P7.62mm_Horizontal, F.Cu at (331.2, 87.4)
- added D42: 1N4148, Diode_THT:D_DO-35_SOD27_P7.62mm_Horizontal, F.Cu at (388.7, 87.4)
- added D43: 1N4148, Diode_THT:D_DO-35_SOD27_P7.62mm_Horizontal, F.Cu at (446.2, 87.4)
- added D44: 1N4148, Diode_THT:D_DO-35_SOD27_P7.62mm_Horizontal, F.Cu at (452.2, 87.4)
- added D45: WS2812B_Unified, chu_main:WS2812D-F5, F.Cu at (159.0, 72.6)
- added D46: WS2812B_Unified, chu_main:WS2812D-F5, F.Cu at (101.0, 72.6)
- added HC-SR04-1: ~, HC-SR04:HC-SR04, F.Cu at (72.0, 88.5)
- added HC-SR04-2: ~, HC-SR04:HC-SR04, F.Cu at (130.0, 88.5)
- added HC-SR04-3: ~, HC-SR04:HC-SR04, F.Cu at (188.0, 88.5)
- added HC-SR04-4: ~, HC-SR04:HC-SR04, F.Cu at (246.0, 88.5)
- added HC-SR04-5: ~, HC-SR04:HC-SR04, F.Cu at (304.0, 88.5)
- added HC-SR04-6: ~, HC-SR04:HC-SR04, F.Cu at (362.0, 88.5)
- added HC-SR04-7: ~, HC-SR04:HC-SR04, F.Cu at (420.0, 88.5)
- added HC-SR04-8: ~, HC-SR04:HC-SR04, F.Cu at (478.0, 88.5)
- added SCR5: ScrewHole, chu_main:MountingHole_3.2mm_M3, F.Cu at (354.6, 205.6)
- added SCR6: ScrewHole, chu_main:MountingHole_3.2mm_M3, F.Cu at (195.4, 205.6)
- added SCR7: ScrewHole, chu_main:MountingHole_3.2mm_M3, F.Cu at (354.0, 66.4)
- added SCR8: ScrewHole, chu_main:MountingHole_3.2mm_M3, F.Cu at (196.0, 66.4)
- D1, D10, D11, D12, D13, D14, D15, D16, D17, D18, D19, D2, D20, D21, D22, D23, D24, D25, D26, D27, D28, D29, D3, D30, D31, D32, D33, D34, D35, D36, D4, D5, D6, D7, D8, D9: footprint chu_main:WS2812B-4020 -> chu_main:WS2812D-F5
- K1, K10, K15, K16, K17, K18, K19, K2, K20, K21, K22, K27, K28, K29, K3, K30, K31, K32, K4, K5, K6, K7, K8, K9: footprint chu_main:ChuKey -> chu_main:Chu_TouchKey
- K11, K14, K23, K26: footprint chu_main:ChuKeyBiasLeft -> chu_main:Chu_TouchKey
- K12, K13, K24, K25: footprint chu_main:ChuKeyBiasRight -> chu_main:Chu_TouchKey
- U2: value PCA9548APW -> SN74LV1T34DBV; footprint Package_SO:TSSOP-24_4.4x7.8mm_P0.65mm -> chu_main:SOT-23-5_Jumper
- moved SCR3 442.9 mm to (512.0, 205.4)
- moved SCR4 322.9 mm to (38.0, 205.4)
- moved K16 285.9 mm to (492.5, 118.0), turned to 0 degrees
- moved K15 259.4 mm to (463.5, 118.0)
- moved K14 242.5 mm to (434.5, 118.0), turned to 0 degrees
- moved K13 216.6 mm to (405.5, 118.0)
- moved K12 199.2 mm to (376.5, 118.0), turned to 0 degrees
- moved K17 181.8 mm to (57.5, 158.5)
- moved SCR2 180.9 mm to (512.0, 66.4)
- moved K32 176.8 mm to (492.5, 158.5), turned to 0 degrees
- moved K11 174.0 mm to (347.5, 118.0)
- moved D31 171.5 mm to (492.5, 93.6), turned to 0 degrees
- moved D30 164.5 mm to (478.0, 93.6), turned to 0 degrees
- moved C7 161.4 mm to (355.7, 95.8)
- moved K31 160.3 mm to (463.5, 158.5)
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Connections:
- D36 pad O: unconnected-(D36-PadO) -> Net-(D36-Out)
- K1 pad 1: Net-(K1-Pad1) -> Net-(K1-Pin_1)
- K10 pad 1: Net-(K10-Pad1) -> Net-(K10-Pin_1)
- K11 pad 1: Net-(K11-Pad1) -> Net-(K11-Pin_1)
- K12 pad 1: Net-(K12-Pad1) -> Net-(K12-Pin_1)
- K13 pad 1: Net-(K13-Pad1) -> Net-(K13-Pin_1)
- K14 pad 1: Net-(K14-Pad1) -> Net-(K14-Pin_1)
- K15 pad 1: Net-(K15-Pad1) -> Net-(K15-Pin_1)
- K16 pad 1: Net-(K16-Pad1) -> Net-(K16-Pin_1)
- K17 pad 1: Net-(K17-Pad1) -> Net-(K17-Pin_1)
- K18 pad 1: Net-(K18-Pad1) -> Net-(K18-Pin_1)
- K19 pad 1: Net-(K19-Pad1) -> Net-(K19-Pin_1)
- K2 pad 1: Net-(K2-Pad1) -> Net-(K2-Pin_1)
- K20 pad 1: Net-(K20-Pad1) -> Net-(K20-Pin_1)
- K21 pad 1: Net-(K21-Pad1) -> Net-(K21-Pin_1)
- K22 pad 1: Net-(K22-Pad1) -> Net-(K22-Pin_1)
- K23 pad 1: Net-(K23-Pad1) -> Net-(K23-Pin_1)
- K24 pad 1: Net-(K24-Pad1) -> Net-(K24-Pin_1)
- K25 pad 1: Net-(K25-Pad1) -> Net-(K25-Pin_1)
- K26 pad 1: Net-(K26-Pad1) -> Net-(K26-Pin_1)
- K27 pad 1: Net-(K27-Pad1) -> Net-(K27-Pin_1)
- K28 pad 1: Net-(K28-Pad1) -> Net-(K28-Pin_1)
- K29 pad 1: Net-(K29-Pad1) -> Net-(K29-Pin_1)
- K3 pad 1: Net-(K3-Pad1) -> Net-(K3-Pin_1)
- K30 pad 1: Net-(K30-Pad1) -> Net-(K30-Pin_1)
- K4 pad 1: Net-(K4-Pad1) -> Net-(K4-Pin_1)
- K5 pad 1: Net-(K5-Pad1) -> Net-(K5-Pin_1)
- K6 pad 1: Net-(K6-Pad1) -> Net-(K6-Pin_1)
- K7 pad 1: Net-(K7-Pad1) -> Net-(K7-Pin_1)
- K8 pad 1: Net-(K8-Pad1) -> Net-(K8-Pin_1)
- K9 pad 1: Net-(K9-Pad1) -> Net-(K9-Pin_1)
- U1 pad 1: unconnected-(U1-Pad1) -> Net-(HC-SR04-1-Trig)
- U1 pad 25: Net-(U1-Pad25) -> unconnected-(U1-GPIO19-Pad25)
- U1 pad 27: unconnected-(U1-Pad27) -> Net-(U1-GPIO21)
- U2 pad 1: GND -> unconnected-(U2-NC-Pad1)
- U2 pad 2: GND -> Net-(D37-A)
- U2 pad 3: Net-(U1-Pad25) -> GND
- U2 pad 4: /SDA_3 -> Net-(U1-GPIO21)
- U2 pad 5: /SCL_3 -> +3V3
- U3 pad 10: Net-(K3-Pad1) -> Net-(K19-Pin_1)
- U3 pad 11: Net-(K4-Pad1) -> Net-(K1-Pin_1)
- U3 pad 12: Net-(K5-Pad1) -> Net-(K2-Pin_1)
- U3 pad 13: Net-(K6-Pad1) -> Net-(K3-Pin_1)
- U3 pad 14: Net-(K7-Pad1) -> Net-(K4-Pin_1)
- U3 pad 15: Net-(K8-Pad1) -> Net-(K5-Pin_1)
- U3 pad 16: Net-(K9-Pad1) -> Net-(K6-Pin_1)
- U3 pad 17: Net-(K10-Pad1) -> Net-(K20-Pin_1)
- U3 pad 18: Net-(K11-Pad1) -> Net-(K21-Pin_1)
- U3 pad 19: Net-(K12-Pad1) -> Net-(K22-Pin_1)
- U3 pad 8: Net-(K1-Pad1) -> Net-(K17-Pin_1)
- U3 pad 9: Net-(K2-Pad1) -> Net-(K18-Pin_1)
- U4 pad 10: Net-(K15-Pad1) -> Net-(K25-Pin_1)
- U4 pad 11: Net-(K16-Pad1) -> Net-(K7-Pin_1)
- U4 pad 12: Net-(K17-Pad1) -> Net-(K8-Pin_1)
- U4 pad 13: Net-(K18-Pad1) -> Net-(K9-Pin_1)
- U4 pad 14: Net-(K19-Pad1) -> Net-(K10-Pin_1)
- U4 pad 15: Net-(K20-Pad1) -> Net-(K11-Pin_1)
- U4 pad 16: Net-(K21-Pad1) -> Net-(K12-Pin_1)
- U4 pad 17: Net-(K22-Pad1) -> Net-(K26-Pin_1)
- U4 pad 18: Net-(K23-Pad1) -> Net-(K27-Pin_1)
- U4 pad 19: Net-(K24-Pad1) -> Net-(K28-Pin_1)
- U4 pad 8: Net-(K13-Pad1) -> Net-(K23-Pin_1)
- U4 pad 9: Net-(K14-Pad1) -> Net-(K24-Pin_1)
- U5 pad 10: Net-(K27-Pad1) -> Net-(K13-Pin_1)
- U5 pad 11: Net-(K28-Pad1) -> Net-(K14-Pin_1)
- U5 pad 12: Net-(K29-Pad1) -> Net-(K15-Pin_1)
- U5 pad 13: Net-(K30-Pad1) -> Net-(K16-Pin_1)
- U5 pad 8: Net-(K25-Pad1) -> Net-(K29-Pin_1)
- U5 pad 9: Net-(K26-Pad1) -> Net-(K30-Pin_1)
Routing:
- net GND: track 167.7 -> 1021.4 mm, vias 48 -> 5
- net +5V: track 761.3 -> 1525.2 mm, vias 14 -> 0
- net Net-(D37-A): track 0.00 -> 583.7 mm, vias 0 -> 4
- net Net-(HC-SR04-1-Trig): track 0.00 -> 550.2 mm, vias 0 -> 2
- net /SDA: track 203.1 -> 378.8 mm, vias 3 -> 0
- net /SCL: track 204.6 -> 373.9 mm, vias 3 -> 0
- net /SDA_5: track 132.0 -> 0.00 mm, vias 1 -> 0
- net /SCL_5: track 129.7 -> 0.00 mm, vias 1 -> 0
- net Net-(K7-Pin_1): track 0.00 -> 110.3 mm, vias 0 -> 1
- net Net-(K6-Pin_1): track 0.00 -> 110.3 mm, vias 0 -> 1
- net Net-(K12-Pin_1): track 0.00 -> 110.2 mm, vias 0 -> 1
- net Net-(K1-Pin_1): track 0.00 -> 109.9 mm, vias 0 -> 1
- net Net-(U1-Pad25): track 97.3 -> 0.00 mm
- net /SDA_1: track 92.6 -> 0.00 mm, vias 3 -> 0
- net /SCL_1: track 89.4 -> 0.00 mm, vias 1 -> 0
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Other:
- board size 294 x 100 mm -> 490 x 155 mm
- board text removed: "Chu Pico V1.5"
